File: 回路/untitled.brd (EAGLE design)
At the start: 93.7 x 92.8 mm, 213 parts, among them Q1 2SJ626, Q2 2SJ626, Q3 BSS138, Q4 BSS138, Q5 2SJ626, Q6 BSS138, Q7 BSS138

Commit message: 仕様追加 　・LINの読み出し追加 　・Orgログ出力フォーマットの変更
Connections:
- removed net N$30: 2-18.1, 2-36.1, JP2.18
- removed net N$69: JP10.7, U$1.P$4
- new net LIN_TX: 2-18.1, 2-36.1, JP10.7, JP2.18
Routing:
- net LIN_TX: track 0.00 -> 35.0 mm, vias 0 -> 1
- net N$69: track 19.9 -> 0.00 mm, vias 1 -> 0
- net N$30: track 15.2 -> 0.00 mm
